File: PCB/MagicBand_Carrier/MagicBand_Carrier.kicad_sch (KiCad schematic)
At the start: 11 parts, among them J1 Pro_Mini_Module, J2 MFRC522_Module, J3 RF_TX_DFLIFE, J4 MOSFET_DRV_IN, J5 MOSFET_DRV_OUT, J6 NeoPixel_Outer_16px, J7 NeoPixel_Inner_12px, J8 PWR_IN_5V, U1 MCP1700-3302

Commit message: Fix undersized MCP1700 decoupling caps per Microchip datasheet
Independent review (separate from the agent that built the schematic)
found C1/C2 both at 100nF. Microchip's DS20001826 specifies 1.0uF as the
standard/minimum output cap for stability -- undersized output
capacitance risks oscillation, and the MFRC522's active-scan current
step (13-26mA) is exactly the kind of load transient that stresses that
margin. C2 (output) -> 1.0uF per datasheet, C1 (input) -> 10uF per
typical reference-design sizing. Re-ran ERC: still 0 errors, same 120
cosmetic warnings.

v2 (PCB/MagicBand_FullyCustom/) doesn't exist yet -- needs the same fix
once it lands.

Co-Authored-By: Claude Sonnet 5 <noreply@anthropic.com>
Parts:
- C1: value 100nF -> 10uF
- C2: value 100nF -> 1.0uF
Changed lines of the file:
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@@
 			(effects (font (size 1.27 1.27)))
 		)
-		(property "Value" "100nF"
+		(property "Value" "10uF"
 			(at 160 101.5 0)
 			(effects (font (size 1.27 1.27)))
@@
 			(effects (font (size 1.27 1.27)))
 		)
-		(property "Value" "100nF"
+		(property "Value" "1.0uF"
 			(at 175 101.5 0)
 			(effects (font (size 1.27 1.27)))
