File: PCB/MagicBand_BarrelJack/MagicBand_BarrelJack.kicad_pcb (KiCad board)
At the start: 2 copper layers, 40 x 40 mm, 20 parts, among them J2 PinSocket_1x08_P2.54mm_Vertic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, J3 PinHeader_1x03_P2.54mm_Vertic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, J6 JST_PH_B3B-PH-K_1x03_P2.00mm_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, J7 JST_PH_B3B-PH-K_1x03_P2.00mm_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, J8 PinHeader_1x02_P2.54mm_Vertic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, J9 PinHeader_2x03_P2.54mm_Vertic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, Q1 SOT-23, U1 DIP-28_W7.62mm, U2 SOT-23, Y1 Crystal_HC49-4H_Vertical

Commit message: Close layout PDR findings: keepout, J9 reposition, mounting holes, silkscreen
Real fixes, honestly reported alongside the DRC delta (139 -> 202
violations -- see PCB Design Plan for full breakdown of why the count
went up despite genuine progress on every item):

- RF antenna keepout properly defined on both copper layers, sized to
  J3's actual footprint + margin; 4 offending track segments (not just
  the 1 originally flagged) rerouted around it
- J9 (ISP header) moved from the wrong side of the board entirely to
  directly adjacent to J2/U1 -- a real placement win, though the manual
  reconnection routing didn't yet capture the benefit (measured trace
  lengths came out longer, not shorter -- reported plainly)
- 3x NPTH mounting holes added, 4.2mm, sized for heat-stake assembly
- All 20 silkscreen reference designators un-hidden
- MFRC522/crystal clearance checked and documented (28.5mm, lower risk
  than flagged, not fully resolvable pre-purchase)

No pcbnew module available in this environment (confirmed) -- all work
done via direct .kicad_pcb editing + kicad-cli DRC validation.

Co-Authored-By: Claude Sonnet 5 <noreply@anthropic.com>
Parts:
- added MH1: MountingHole_4.2mm, MountingHole:MountingHole_4.2mm, F.Cu at (3.00, 37.0)
- added MH2: MountingHole_4.2mm, MountingHole:MountingHole_4.2mm, F.Cu at (37.0, 37.0)
- added MH3: MountingHole_4.2mm, MountingHole:MountingHole_4.2mm, F.Cu at (37.0, 20.0)
- moved J9 34.0 mm to (10.5, 10.0)
Routing:
- net MCU_RESET: track 26.4 -> 51.4 mm
- net D12: track 51.4 -> 73.4 mm
- net +5V: track 97.2 -> 118.3 mm
- net D13: track 59.0 -> 74.9 mm
- net D11: track 59.0 -> 69.9 mm
- net +3V3: track 77.1 -> 83.8 mm

Commit message: Remove J7 (inner NeoPixel ring) from schematic and PCB, verified clean
Completes the LED-strip scope change deferred at the end of the last
session. Removed J7 (component, D6 wiring, its dedicated power
symbols) from the schematic, its footprint plus 2 dangling track
stubs from the PCB, and renamed J6's value to NeoPixel_LED_Strip
(count-agnostic, pending the ordered strip).

Verified via kicad-cli, not assumed: ERC 0 errors (129 warnings, down
from 209, all pre-existing cosmetic), DRC 0 unconnected pads / 0
footprint errors (188 violations, down from 202). Confirmed side
benefit: npth_inside_courtyard dropped 3->2, the MH3/J7 courtyard
conflict is gone. Regenerated all tracked exports (ERC/DRC reports,
schematic PDF, board SVGs) to match.

Co-Authored-By: Claude Sonnet 5 <noreply@anthropic.com>
Claude-Session: https://claude.ai/code/session_01WRfsGJdmccHFit2MbdKbSy
Parts:
- removed J7: JST_PH_B3B-PH-K_1x03_P2.00mm_Vertical, JST_PH_B3B-PH-K_1x03_P2.00mm_Vertical
Routing:
- net D6: track 30.4 -> 0.00 mm

Commit message: Finalize PCB placement: fix MH3/J6 courtyard conflict, silkscreen label overlaps
Moves MH3 clear of J6's courtyard (the one error-level placement issue),
nudges R1/C4 reference fields off neighboring silkscreen/pads. Net DRC:
188 -> 176 violations. U2/J2 label overlap left open, needs GUI (see
Session Log). Also stashed a stale-base uncommitted change found in the
main checkout and logged a PM process suggestion about pulling before
trusting local git state.

Co-Authored-By: Claude Sonnet 5 <noreply@anthropic.com>
Claude-Session: https://claude.ai/code/session_01UiULxbNnG293uuE4csn9nG
Parts:
- moved MH3 7.00 mm to (37.0, 27.0)
Changed lines of the file:
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@@
 		(tags "capacitor")
 		(property "Reference" "C4"
-			(at 0 -1.43 0)
+			(at 0 1.43 0)
 			(layer "F.SilkS")
 			(effects
@@
 		(tags "resistor")
 		(property "Reference" "R1"
-			(at 0 -1.43 0)
+			(at 2.2 0 0)
 			(layer "F.SilkS")
 			(effects
@@
 	(footprint "MountingHole:MountingHole_4.2mm"
 		(layer "F.Cu")
-		(at 37 20)
+		(at 37 27)
 		(descr "Mounting Hole 4.2mm, no annular ring -- heat-stake, non-plated")
 		(tags "mounting hole")
